Commit message: First env version

File: assets/drone.xacro (robot description, xacro)
@@ -114,31 +114,31 @@
             </inertial>
         </link>
-        <joint name="${prefix}_prop1joint" type="continous">
+        <joint name="${prefix}_prop1joint" type="fixed">
             <parent link="${prefix}_base" />
             <child link="${prefix}_prop1" />
-            <limit effort="3000" velocity="10000.0"/>
             <origin xyz="${arm_x} ${arm_y} 0.04" rpy="0 0 0" />
-            <axis xyz="0 0 1" />
+            <!--<limit effort="3000" velocity="10000.0"/>
+            <axis xyz="0 0 1" />-->
         </joint>
-        <joint name="${prefix}_prop2joint" type="continous">
+        <joint name="${prefix}_prop2joint" type="fixed">
             <parent link="${prefix}_base" />
             <child link="${prefix}_prop2" />
-            <limit effort="3000" velocity="10000.0"/>
             <origin xyz="${-arm_x} ${arm_y} 0.04" rpy="0 0 0" />
-            <axis xyz="0 0 1" />
+            <!--<limit effort="3000" velocity="10000.0"/>
+            <axis xyz="0 0 1" />-->
         </joint>
-        <joint name="${prefix}_prop3joint" type="continous">
+        <joint name="${prefix}_prop3joint" type="fixed">
             <parent link="${prefix}_base" />
             <child link="${prefix}_prop3" />
-            <limit effort="3000" velocity="10000.0"/>
             <origin xyz="${-arm_x} ${-arm_y} 0.04" rpy="0 0 0" />
-            <axis xyz="0 0 1" />
+            <!--<limit effort="3000" velocity="10000.0"/>
+            <axis xyz="0 0 1" />-->
         </joint>
-        <joint name="${prefix}_prop4joint" type="continous">
+        <joint name="${prefix}_prop4joint" type="fixed">
             <parent link="${prefix}_base" />
             <child link="${prefix}_prop4" />
-            <limit effort="3000" velocity="10000.0"/>
             <origin xyz="${arm_x} ${-arm_y} 0.04" rpy="0 0 0" />
-            <axis xyz="0 0 1" />
+            <!--<limit effort="3000" velocity="10000.0"/>
+            <axis xyz="0 0 1" />-->
         </joint>
     </xacro:macro>

File: assets/drone_w_arms.urdf (robot description, URDF)
Before this commit: robot drone_w_arms, 25 links, 20 joints
Links:
- added link arm1_link_10, mass 0.009090909090909092; collision cylinder length=0.03 radius=0.01; visual mesh filename=meshes/single_segment.dae scale=0.0006 0.0006 0.00030000000000000003
- added link arm1_link_3, mass 0.009090909090909092; collision cylinder length=0.03 radius=0.01; visual mesh filename=meshes/single_segment.dae scale=0.0006 0.0006 0.00030000000000000003
- added link arm1_link_4, mass 0.009090909090909092; collision cylinder length=0.03 radius=0.01; visual mesh filename=meshes/single_segment.dae scale=0.0006 0.0006 0.00030000000000000003
- added link arm1_link_5, mass 0.009090909090909092; collision cylinder length=0.03 radius=0.01; visual mesh filename=meshes/single_segment.dae scale=0.0006 0.0006 0.00030000000000000003
- added link arm1_link_6, mass 0.009090909090909092; collision cylinder length=0.03 radius=0.01; visual mesh filename=meshes/single_segment.dae scale=0.0006 0.0006 0.00030000000000000003
- added link arm1_link_7, mass 0.009090909090909092; collision cylinder length=0.03 radius=0.01; visual mesh filename=meshes/single_segment.dae scale=0.0006 0.0006 0.00030000000000000003
- added link arm1_link_8, mass 0.009090909090909092; collision cylinder length=0.03 radius=0.01; visual mesh filename=meshes/single_segment.dae scale=0.0006 0.0006 0.00030000000000000003
- added link arm1_link_9, mass 0.009090909090909092; collision cylinder length=0.03 radius=0.01; visual mesh filename=meshes/single_segment.dae scale=0.0006 0.0006 0.00030000000000000003
- added link arm2_link_10, mass 0.009090909090909092; collision cylinder length=0.03 radius=0.01; visual mesh filename=meshes/single_segment.dae scale=0.0006 0.0006 0.00030000000000000003
- added link arm2_link_3, mass 0.009090909090909092; collision cylinder length=0.03 radius=0.01; visual mesh filename=meshes/single_segment.dae scale=0.0006 0.0006 0.00030000000000000003
- added link arm2_link_4, mass 0.009090909090909092; collision cylinder length=0.03 radius=0.01; visual mesh filename=meshes/single_segment.dae scale=0.0006 0.0006 0.00030000000000000003
- added link arm2_link_5, mass 0.009090909090909092; collision cylinder length=0.03 radius=0.01; visual mesh filename=meshes/single_segment.dae scale=0.0006 0.0006 0.00030000000000000003
- added link arm2_link_6, mass 0.009090909090909092; collision cylinder length=0.03 radius=0.01; visual mesh filename=meshes/single_segment.dae scale=0.0006 0.0006 0.00030000000000000003
- added link arm2_link_7, mass 0.009090909090909092; collision cylinder length=0.03 radius=0.01; visual mesh filename=meshes/single_segment.dae scale=0.0006 0.0006 0.00030000000000000003
- added link arm2_link_8, mass 0.009090909090909092; collision cylinder length=0.03 radius=0.01; visual mesh filename=meshes/single_segment.dae scale=0.0006 0.0006 0.00030000000000000003
- added link arm2_link_9, mass 0.009090909090909092; collision cylinder length=0.03 radius=0.01; visual mesh filename=meshes/single_segment.dae scale=0.0006 0.0006 0.00030000000000000003
- added link arm3_link_10, mass 0.009090909090909092; collision cylinder length=0.03 radius=0.01; visual mesh filename=meshes/single_segment.dae scale=0.0006 0.0006 0.00030000000000000003
- added link arm3_link_3, mass 0.009090909090909092; collision cylinder length=0.03 radius=0.01; visual mesh filename=meshes/single_segment.dae scale=0.0006 0.0006 0.00030000000000000003
- added link arm3_link_4, mass 0.009090909090909092; collision cylinder length=0.03 radius=0.01; visual mesh filename=meshes/single_segment.dae scale=0.0006 0.0006 0.00030000000000000003
- added link arm3_link_5, mass 0.009090909090909092; collision cylinder length=0.03 radius=0.01; visual mesh filename=meshes/single_segment.dae scale=0.0006 0.0006 0.00030000000000000003
- added link arm3_link_6, mass 0.009090909090909092; collision cylinder length=0.03 radius=0.01; visual mesh filename=meshes/single_segment.dae scale=0.0006 0.0006 0.00030000000000000003
- added link arm3_link_7, mass 0.009090909090909092; collision cylinder length=0.03 radius=0.01; visual mesh filename=meshes/single_segment.dae scale=0.0006 0.0006 0.00030000000000000003
- added link arm3_link_8, mass 0.009090909090909092; collision cylinder length=0.03 radius=0.01; visual mesh filename=meshes/single_segment.dae scale=0.0006 0.0006 0.00030000000000000003
- added link arm3_link_9, mass 0.009090909090909092; collision cylinder length=0.03 radius=0.01; visual mesh filename=meshes/single_segment.dae scale=0.0006 0.0006 0.00030000000000000003
- added link arm4_link_10, mass 0.009090909090909092; collision cylinder length=0.03 radius=0.01; visual mesh filename=meshes/single_segment.dae scale=0.0006 0.0006 0.00030000000000000003
- added link arm4_link_3, mass 0.009090909090909092; collision cylinder length=0.03 radius=0.01; visual mesh filename=meshes/single_segment.dae scale=0.0006 0.0006 0.00030000000000000003
- added link arm4_link_4, mass 0.009090909090909092; collision cylinder length=0.03 radius=0.01; visual mesh filename=meshes/single_segment.dae scale=0.0006 0.0006 0.00030000000000000003
- added link arm4_link_5, mass 0.009090909090909092; collision cylinder length=0.03 radius=0.01; visual mesh filename=meshes/single_segment.dae scale=0.0006 0.0006 0.00030000000000000003
- added link arm4_link_6, mass 0.009090909090909092; collision cylinder length=0.03 radius=0.01; visual mesh filename=meshes/single_segment.dae scale=0.0006 0.0006 0.00030000000000000003
- added link arm4_link_7, mass 0.009090909090909092; collision cylinder length=0.03 radius=0.01; visual mesh filename=meshes/single_segment.dae scale=0.0006 0.0006 0.00030000000000000003
- added link arm4_link_8, mass 0.009090909090909092; collision cylinder length=0.03 radius=0.01; visual mesh filename=meshes/single_segment.dae scale=0.0006 0.0006 0.00030000000000000003
- added link arm4_link_9, mass 0.009090909090909092; collision cylinder length=0.03 radius=0.01; visual mesh filename=meshes/single_segment.dae scale=0.0006 0.0006 0.00030000000000000003
- link arm1_link_1: mass 0.3333333333333333 -> 0.009090909090909092; geometry collision cylinder length=0.03 radius=0.01; visual mesh filename=meshes/single_segment.dae scale=0.0006 0.0006 0.00030000000000000003
- link arm1_link_2: mass 0.3333333333333333 -> 0.009090909090909092; geometry collision cylinder length=0.03 radius=0.01; visual mesh filename=meshes/single_segment.dae scale=0.0006 0.0006 0.00030000000000000003
- link arm1_sphere: mass 0.3333333333333333 -> 0.009090909090909092
- link arm2_link_1: mass 0.3333333333333333 -> 0.009090909090909092; geometry collision cylinder length=0.03 radius=0.01; visual mesh filename=meshes/single_segment.dae scale=0.0006 0.0006 0.00030000000000000003
- link arm2_link_2: mass 0.3333333333333333 -> 0.009090909090909092; geometry collision cylinder length=0.03 radius=0.01; visual mesh filename=meshes/single_segment.dae scale=0.0006 0.0006 0.00030000000000000003
- link arm2_sphere: mass 0.3333333333333333 -> 0.009090909090909092
- link arm3_link_1: mass 0.3333333333333333 -> 0.009090909090909092; geometry collision cylinder length=0.03 radius=0.01; visual mesh filename=meshes/single_segment.dae scale=0.0006 0.0006 0.00030000000000000003
- link arm3_link_2: mass 0.3333333333333333 -> 0.009090909090909092; geometry collision cylinder length=0.03 radius=0.01; visual mesh filename=meshes/single_segment.dae scale=0.0006 0.0006 0.00030000000000000003
- link arm3_sphere: mass 0.3333333333333333 -> 0.009090909090909092
- link arm4_link_1: mass 0.3333333333333333 -> 0.009090909090909092; geometry collision cylinder length=0.03 radius=0.01; visual mesh filename=meshes/single_segment.dae scale=0.0006 0.0006 0.00030000000000000003
- link arm4_link_2: mass 0.3333333333333333 -> 0.009090909090909092; geometry collision cylinder length=0.03 radius=0.01; visual mesh filename=meshes/single_segment.dae scale=0.0006 0.0006 0.00030000000000000003
- link arm4_sphere: mass 0.3333333333333333 -> 0.009090909090909092
Joints:
- added joint arm1_joint: type fixed, parent drone_base, child arm1_base
- added joint arm1_joint_10: type revolute, parent arm1_link_9, child arm1_link_10, origin xyz=0 0 0.03 rpy=0 0 0, axis 1 0 0, limit lower=-1.57 upper=1.57 effort=10.0 velocity=1.0
- added joint arm1_joint_3: type revolute, parent arm1_link_2, child arm1_link_3, origin xyz=0 0 0.03 rpy=0 0 0, axis 1 0 0, limit lower=-1.57 upper=1.57 effort=10.0 velocity=1.0
- added joint arm1_joint_4: type revolute, parent arm1_link_3, child arm1_link_4, origin xyz=0 0 0.03 rpy=0 0 0, axis 1 0 0, limit lower=-1.57 upper=1.57 effort=10.0 velocity=1.0
- added joint arm1_joint_5: type revolute, parent arm1_link_4, child arm1_link_5, origin xyz=0 0 0.03 rpy=0 0 0, axis 1 0 0, limit lower=-1.57 upper=1.57 effort=10.0 velocity=1.0
- added joint arm1_joint_6: type revolute, parent arm1_link_5, child arm1_link_6, origin xyz=0 0 0.03 rpy=0 0 0, axis 1 0 0, limit lower=-1.57 upper=1.57 effort=10.0 velocity=1.0
- added joint arm1_joint_7: type revolute, parent arm1_link_6, child arm1_link_7, origin xyz=0 0 0.03 rpy=0 0 0, axis 1 0 0, limit lower=-1.57 upper=1.57 effort=10.0 velocity=1.0
- added joint arm1_joint_8: type revolute, parent arm1_link_7, child arm1_link_8, origin xyz=0 0 0.03 rpy=0 0 0, axis 1 0 0, limit lower=-1.57 upper=1.57 effort=10.0 velocity=1.0
- added joint arm1_joint_9: type revolute, parent arm1_link_8, child arm1_link_9, origin xyz=0 0 0.03 rpy=0 0 0, axis 1 0 0, limit lower=-1.57 upper=1.57 effort=10.0 velocity=1.0
- added joint arm2_joint: type fixed, parent drone_base, child arm2_base
- added joint arm2_joint_10: type revolute, parent arm2_link_9, child arm2_link_10, origin xyz=0 0 0.03 rpy=0 0 0, axis 1 0 0, limit lower=-1.57 upper=1.57 effort=10.0 velocity=1.0
- added joint arm2_joint_3: type revolute, parent arm2_link_2, child arm2_link_3, origin xyz=0 0 0.03 rpy=0 0 0, axis 1 0 0, limit lower=-1.57 upper=1.57 effort=10.0 velocity=1.0
- added joint arm2_joint_4: type revolute, parent arm2_link_3, child arm2_link_4, origin xyz=0 0 0.03 rpy=0 0 0, axis 1 0 0, limit lower=-1.57 upper=1.57 effort=10.0 velocity=1.0
- added joint arm2_joint_5: type revolute, parent arm2_link_4, child arm2_link_5, origin xyz=0 0 0.03 rpy=0 0 0, axis 1 0 0, limit lower=-1.57 upper=1.57 effort=10.0 velocity=1.0
- added joint arm2_joint_6: type revolute, parent arm2_link_5, child arm2_link_6, origin xyz=0 0 0.03 rpy=0 0 0, axis 1 0 0, limit lower=-1.57 upper=1.57 effort=10.0 velocity=1.0
- added joint arm2_joint_7: type revolute, parent arm2_link_6, child arm2_link_7, origin xyz=0 0 0.03 rpy=0 0 0, axis 1 0 0, limit lower=-1.57 upper=1.57 effort=10.0 velocity=1.0
- added joint arm2_joint_8: type revolute, parent arm2_link_7, child arm2_link_8, origin xyz=0 0 0.03 rpy=0 0 0, axis 1 0 0, limit lower=-1.57 upper=1.57 effort=10.0 velocity=1.0
- added joint arm2_joint_9: type revolute, parent arm2_link_8, child arm2_link_9, origin xyz=0 0 0.03 rpy=0 0 0, axis 1 0 0, limit lower=-1.57 upper=1.57 effort=10.0 velocity=1.0
- added joint arm3_joint: type fixed, parent drone_base, child arm3_base
- added joint arm3_joint_10: type revolute, parent arm3_link_9, child arm3_link_10, origin xyz=0 0 0.03 rpy=0 0 0, axis 1 0 0, limit lower=-1.57 upper=1.57 effort=10.0 velocity=1.0
- added joint arm3_joint_3: type revolute, parent arm3_link_2, child arm3_link_3, origin xyz=0 0 0.03 rpy=0 0 0, axis 1 0 0, limit lower=-1.57 upper=1.57 effort=10.0 velocity=1.0
- added joint arm3_joint_4: type revolute, parent arm3_link_3, child arm3_link_4, origin xyz=0 0 0.03 rpy=0 0 0, axis 1 0 0, limit lower=-1.57 upper=1.57 effort=10.0 velocity=1.0
- added joint arm3_joint_5: type revolute, parent arm3_link_4, child arm3_link_5, origin xyz=0 0 0.03 rpy=0 0 0, axis 1 0 0, limit lower=-1.57 upper=1.57 effort=10.0 velocity=1.0
- added joint arm3_joint_6: type revolute, parent arm3_link_5, child arm3_link_6, origin xyz=0 0 0.03 rpy=0 0 0, axis 1 0 0, limit lower=-1.57 upper=1.57 effort=10.0 velocity=1.0
- added joint arm3_joint_7: type revolute, parent arm3_link_6, child arm3_link_7, origin xyz=0 0 0.03 rpy=0 0 0, axis 1 0 0, limit lower=-1.57 upper=1.57 effort=10.0 velocity=1.0
- added joint arm3_joint_8: type revolute, parent arm3_link_7, child arm3_link_8, origin xyz=0 0 0.03 rpy=0 0 0, axis 1 0 0, limit lower=-1.57 upper=1.57 effort=10.0 velocity=1.0
- added joint arm3_joint_9: type revolute, parent arm3_link_8, child arm3_link_9, origin xyz=0 0 0.03 rpy=0 0 0, axis 1 0 0, limit lower=-1.57 upper=1.57 effort=10.0 velocity=1.0
- added joint arm4_joint: type fixed, parent drone_base, child arm4_base
- added joint arm4_joint_10: type revolute, parent arm4_link_9, child arm4_link_10, origin xyz=0 0 0.03 rpy=0 0 0, axis 1 0 0, limit lower=-1.57 upper=1.57 effort=10.0 velocity=1.0
- added joint arm4_joint_3: type revolute, parent arm4_link_2, child arm4_link_3, origin xyz=0 0 0.03 rpy=0 0 0, axis 1 0 0, limit lower=-1.57 upper=1.57 effort=10.0 velocity=1.0
- added joint arm4_joint_4: type revolute, parent arm4_link_3, child arm4_link_4, origin xyz=0 0 0.03 rpy=0 0 0, axis 1 0 0, limit lower=-1.57 upper=1.57 effort=10.0 velocity=1.0
- added joint arm4_joint_5: type revolute, parent arm4_link_4, child arm4_link_5, origin xyz=0 0 0.03 rpy=0 0 0, axis 1 0 0, limit lower=-1.57 upper=1.57 effort=10.0 velocity=1.0
- added joint arm4_joint_6: type revolute, parent arm4_link_5, child arm4_link_6, origin xyz=0 0 0.03 rpy=0 0 0, axis 1 0 0, limit lower=-1.57 upper=1.57 effort=10.0 velocity=1.0
- added joint arm4_joint_7: type revolute, parent arm4_link_6, child arm4_link_7, origin xyz=0 0 0.03 rpy=0 0 0, axis 1 0 0, limit lower=-1.57 upper=1.57 effort=10.0 velocity=1.0
- added joint arm4_joint_8: type revolute, parent arm4_link_7, child arm4_link_8, origin xyz=0 0 0.03 rpy=0 0 0, axis 1 0 0, limit lower=-1.57 upper=1.57 effort=10.0 velocity=1.0
- added joint arm4_joint_9: type revolute, parent arm4_link_8, child arm4_link_9, origin xyz=0 0 0.03 rpy=0 0 0, axis 1 0 0, limit lower=-1.57 upper=1.57 effort=10.0 velocity=1.0
- joint arm1_fixed_joint_sphere: origin xyz=0 0 0.13999999999999999 rpy=0 0 0 -> xyz=0 0 0.019999999999999997 rpy=0 0 0; parent arm1_link_2 -> arm1_link_10
- joint arm1_joint_2: origin xyz=0 0 0.15 rpy=0 0 0 -> xyz=0 0 0.03 rpy=0 0 0
- joint arm2_fixed_joint_sphere: origin xyz=0 0 0.13999999999999999 rpy=0 0 0 -> xyz=0 0 0.019999999999999997 rpy=0 0 0; parent arm2_link_2 -> arm2_link_10
- joint arm2_joint_2: origin xyz=0 0 0.15 rpy=0 0 0 -> xyz=0 0 0.03 rpy=0 0 0
- joint arm3_fixed_joint_sphere: origin xyz=0 0 0.13999999999999999 rpy=0 0 0 -> xyz=0 0 0.019999999999999997 rpy=0 0 0; parent arm3_link_2 -> arm3_link_10
- joint arm3_joint_2: origin xyz=0 0 0.15 rpy=0 0 0 -> xyz=0 0 0.03 rpy=0 0 0
- joint arm4_fixed_joint_sphere: origin xyz=0 0 0.13999999999999999 rpy=0 0 0 -> xyz=0 0 0.019999999999999997 rpy=0 0 0; parent arm4_link_2 -> arm4_link_10
- joint arm4_joint_2: origin xyz=0 0 0.15 rpy=0 0 0 -> xyz=0 0 0.03 rpy=0 0 0
- joint drone_prop1joint: axis 0 0 1 -> (none); limit effort=3000 velocity=10000.0 -> (none); type continous -> fixed
- joint drone_prop2joint: axis 0 0 1 -> (none); limit effort=3000 velocity=10000.0 -> (none); type continous -> fixed
- joint drone_prop3joint: axis 0 0 1 -> (none); limit effort=3000 velocity=10000.0 -> (none); type continous -> fixed
- joint drone_prop4joint: axis 0 0 1 -> (none); limit effort=3000 velocity=10000.0 -> (none); type continous -> fixed
- joint x_pos: limit lower=-1 upper=1 effort=100 velocity=100 -> lower=-100 upper=100 effort=100 velocity=100
- joint y_pos: limit lower=-1 upper=1 effort=100 velocity=100 -> lower=-100 upper=100 effort=100 velocity=100
- joint z_pos: limit lower=-1 upper=1 effort=100 velocity=100 -> lower=-100 upper=100 effort=100 velocity=100

File: assets/drone_w_arms.xacro (robot description, xacro)
@@ -1,6 +1,6 @@
 <?xml version="1.0"?>
 <robot xmlns:xacro="http://www.ros.org/wiki/xacro" name="drone_w_arms">
-    <xacro:property name="min_ax" value="-1"/>
-    <xacro:property name="max_ax" value="1"/>
+    <xacro:property name="min_ax" value="-100"/>
+    <xacro:property name="max_ax" value="100"/>
     <!-- Include the robot macro -->
     <xacro:include filename="drone.xacro"/>
@@ -8,9 +8,4 @@
     <!-- Add Drone Base -->
     <xacro:drone_base prefix="drone"/>
-    <!-- Add dummy arms -->
-    <xacro:flex_arm prefix="arm1" L="0.3" n="10" m="1.0" xyz=" 0.175  0.175 0" rpy="3.141 0 -0.7854"/>
-    <xacro:flex_arm prefix="arm2" L="0.3" n="10" m="1.0" xyz=" 0.175 -0.175 0" rpy="3.141 0 -2.3562"/>
-    <xacro:flex_arm prefix="arm3" L="0.3" n="10" m="1.0" xyz="-0.175 -0.175 0" rpy="3.141 0 2.3562"/>
-    <xacro:flex_arm prefix="arm4" L="0.3" n="10" m="1.0" xyz="-0.175  0.175 0" rpy="3.141 0 0.7854"/>
     <!-- Define dummy links for motion generation -->
     <link name="world"/>
@@ -42,3 +37,24 @@
         <dynamics damping="100.0" friction="0.0"/>
     </joint>
+    <!-- Add dummy arms -->
+    <xacro:flex_arm prefix="arm1" L="0.3" n="10" m="0.1" xyz=" 0.175  0.175 0" rpy="3.141 0 -0.7854"/>
+    <xacro:flex_arm prefix="arm2" L="0.3" n="10" m="0.1" xyz=" 0.175 -0.175 0" rpy="3.141 0 -2.3562"/>
+    <xacro:flex_arm prefix="arm3" L="0.3" n="10" m="0.1" xyz="-0.175 -0.175 0" rpy="3.141 0 2.3562"/>
+    <xacro:flex_arm prefix="arm4" L="0.3" n="10" m="0.1" xyz="-0.175  0.175 0" rpy="3.141 0 0.7854"/>
+    <joint name="arm1_joint" type="fixed">
+        <parent link="drone_base"/>
+        <child link="arm1_base" />
+    </joint>
+    <joint name="arm2_joint" type="fixed">
+        <parent link="drone_base"/>
+        <child link="arm2_base" />
+    </joint>
+    <joint name="arm3_joint" type="fixed">
+        <parent link="drone_base"/>
+        <child link="arm3_base" />
+    </joint>
+    <joint name="arm4_joint" type="fixed">
+        <parent link="drone_base"/>
+        <child link="arm4_base" />
+    </joint>
 </robot>

File: assets/dummy_arm.xacro (robot description, xacro)
@@ -28,5 +28,5 @@
             <visual>
                 <geometry>
-                    <mesh filename="./meshes/single_segment.dae" scale="0.0006 0.0006 ${0.003 / n}"/>
+                    <mesh filename="meshes/single_segment.dae" scale="0.0006 0.0006 ${0.003 / n}"/>
                 </geometry>
                 <origin xyz="0 0 ${l / 2}" />
@@ -62,5 +62,5 @@
                 <visual>
                     <geometry>
-                        <mesh filename="./meshes/single_segment.dae" scale="0.0006 0.0006 ${0.003 / N}"/>
+                        <mesh filename="meshes/single_segment.dae" scale="0.0006 0.0006 ${0.003 / N}"/>
                     </geometry>
                     <origin xyz="0 0 ${l / 2}" />

Commit message: Fix collision sizes

File: assets/drone.xacro (robot description, xacro)
@@ -2,6 +2,6 @@
 <robot xmlns:xacro="http://www.ros.org/wiki/xacro">
     <xacro:property name="pi2" value="${pi * 0.5}" />
-    <xacro:property name="l1" value="0.625" />
-    <xacro:property name="l2" value="0.625" />
+    <xacro:property name="l1" value="0.525" />
+    <xacro:property name="l2" value="0.525" />
     <xacro:property name="l3" value="0.1" />
     <xacro:property name="arm_x" value="0.175"/>

File: assets/drone_w_arms.urdf (robot description, URDF)
Before this commit: robot drone_w_arms, 57 links, 56 joints
Links:
- link drone_base: geometry collision box size=0.525 0.525 0.1; visual mesh filename=./meshes/Holybro-X500-V2-no-landinggear-arm-attachments.dae
