Commit message: Fix exploding position bug and make debug errors work for many envs

File: assets/drone.xacro (robot description, xacro)
@@ -7,5 +7,5 @@
     <xacro:property name="arm_x" value="0.175"/>
     <xacro:property name="arm_y" value="0.175"/>
-    <xacro:property name="m" value="1" />
+    <xacro:property name="m" value="10.0" />
     <xacro:macro name="box_inertia" params="l1 l2 l3 mass">
         <inertia ixx="${1/12*mass*(l3*l3 + l1*l1)}" ixy="0.0" ixz="0.0"

File: assets/drone_w_arms.urdf (robot description, URDF)
Before this commit: robot drone_w_arms, 57 links, 56 joints
Links:
- link arm1_link_1: mass 0.009090909090909092 -> 0.09090909090909091
- link arm1_link_10: mass 0.009090909090909092 -> 0.09090909090909091
- link arm1_link_2: mass 0.009090909090909092 -> 0.09090909090909091
- link arm1_link_3: mass 0.009090909090909092 -> 0.09090909090909091
- link arm1_link_4: mass 0.009090909090909092 -> 0.09090909090909091
- link arm1_link_5: mass 0.009090909090909092 -> 0.09090909090909091
- link arm1_link_6: mass 0.009090909090909092 -> 0.09090909090909091
- link arm1_link_7: mass 0.009090909090909092 -> 0.09090909090909091
- link arm1_link_8: mass 0.009090909090909092 -> 0.09090909090909091
- link arm1_link_9: mass 0.009090909090909092 -> 0.09090909090909091
- link arm1_sphere: mass 0.009090909090909092 -> 0.09090909090909091
- link arm2_link_1: mass 0.009090909090909092 -> 0.09090909090909091
- link arm2_link_10: mass 0.009090909090909092 -> 0.09090909090909091
- link arm2_link_2: mass 0.009090909090909092 -> 0.09090909090909091
- link arm2_link_3: mass 0.009090909090909092 -> 0.09090909090909091
- link arm2_link_4: mass 0.009090909090909092 -> 0.09090909090909091
- link arm2_link_5: mass 0.009090909090909092 -> 0.09090909090909091
- link arm2_link_6: mass 0.009090909090909092 -> 0.09090909090909091
- link arm2_link_7: mass 0.009090909090909092 -> 0.09090909090909091
- link arm2_link_8: mass 0.009090909090909092 -> 0.09090909090909091
- link arm2_link_9: mass 0.009090909090909092 -> 0.09090909090909091
- link arm2_sphere: mass 0.009090909090909092 -> 0.09090909090909091
- link arm3_link_1: mass 0.009090909090909092 -> 0.09090909090909091
- link arm3_link_10: mass 0.009090909090909092 -> 0.09090909090909091
- link arm3_link_2: mass 0.009090909090909092 -> 0.09090909090909091
- link arm3_link_3: mass 0.009090909090909092 -> 0.09090909090909091
- link arm3_link_4: mass 0.009090909090909092 -> 0.09090909090909091
- link arm3_link_5: mass 0.009090909090909092 -> 0.09090909090909091
- link arm3_link_6: mass 0.009090909090909092 -> 0.09090909090909091
- link arm3_link_7: mass 0.009090909090909092 -> 0.09090909090909091
- link arm3_link_8: mass 0.009090909090909092 -> 0.09090909090909091
- link arm3_link_9: mass 0.009090909090909092 -> 0.09090909090909091
- link arm3_sphere: mass 0.009090909090909092 -> 0.09090909090909091
- link arm4_link_1: mass 0.009090909090909092 -> 0.09090909090909091
- link arm4_link_10: mass 0.009090909090909092 -> 0.09090909090909091
- link arm4_link_2: mass 0.009090909090909092 -> 0.09090909090909091
- link arm4_link_3: mass 0.009090909090909092 -> 0.09090909090909091
- link arm4_link_4: mass 0.009090909090909092 -> 0.09090909090909091
- link arm4_link_5: mass 0.009090909090909092 -> 0.09090909090909091
- link arm4_link_6: mass 0.009090909090909092 -> 0.09090909090909091
- link arm4_link_7: mass 0.009090909090909092 -> 0.09090909090909091
- link arm4_link_8: mass 0.009090909090909092 -> 0.09090909090909091
- link arm4_link_9: mass 0.009090909090909092 -> 0.09090909090909091
- link arm4_sphere: mass 0.009090909090909092 -> 0.09090909090909091
- link drone_base: mass 1 -> 10.0
Joints:
- joint x_pos: limit lower=-100 upper=100 effort=100 velocity=100 -> lower=-1000 upper=1000 effort=1000 velocity=1000
- joint y_pos: limit lower=-100 upper=100 effort=100 velocity=100 -> lower=-1000 upper=1000 effort=1000 velocity=1000
- joint z_pos: limit lower=-100 upper=100 effort=100 velocity=100 -> lower=-1000 upper=1000 effort=1000 velocity=1000

File: assets/drone_w_arms.xacro (robot description, xacro)
@@ -1,6 +1,6 @@
 <?xml version="1.0"?>
 <robot xmlns:xacro="http://www.ros.org/wiki/xacro" name="drone_w_arms">
-    <xacro:property name="min_ax" value="-100"/>
-    <xacro:property name="max_ax" value="100"/>
+    <xacro:property name="min_ax" value="-1000"/>
+    <xacro:property name="max_ax" value="1000"/>
     <!-- Include the robot macro -->
     <xacro:include filename="drone.xacro"/>
@@ -17,5 +17,5 @@
         <child link="p1" />
         <axis xyz="1 0 0"/>
-        <limit lower="${min_ax}" upper="${max_ax}" effort="100" velocity="100"/>
+        <limit lower="${min_ax}" upper="${max_ax}" effort="1000" velocity="1000"/>
     </joint>
     <joint name="y_pos" type="prismatic">
@@ -23,5 +23,5 @@
         <child link="p2" />
         <axis xyz="0 1 0"/>
-        <limit lower="${min_ax}" upper="${max_ax}" effort="100" velocity="100"/>
+        <limit lower="${min_ax}" upper="${max_ax}" effort="1000" velocity="1000"/>
     </joint>
     <joint name="z_pos" type="prismatic">
@@ -29,5 +29,5 @@
         <child link="p3" />
         <axis xyz="0 0 1"/>
-        <limit lower="${min_ax}" upper="${max_ax}" effort="100" velocity="100"/>
+        <limit lower="${min_ax}" upper="${max_ax}" effort="1000" velocity="1000"/>
     </joint>
     <joint name="base_joint" type="continuous">
@@ -38,8 +38,8 @@
     </joint>
     <!-- Add dummy arms -->
-    <xacro:flex_arm prefix="arm1" L="0.3" n="10" m="0.1" xyz=" 0.175  0.175 0" rpy="3.141 0 -0.7854"/>
-    <xacro:flex_arm prefix="arm2" L="0.3" n="10" m="0.1" xyz=" 0.175 -0.175 0" rpy="3.141 0 -2.3562"/>
-    <xacro:flex_arm prefix="arm3" L="0.3" n="10" m="0.1" xyz="-0.175 -0.175 0" rpy="3.141 0 2.3562"/>
-    <xacro:flex_arm prefix="arm4" L="0.3" n="10" m="0.1" xyz="-0.175  0.175 0" rpy="3.141 0 0.7854"/>
+    <xacro:flex_arm prefix="arm1" L="0.3" n="10" m="1.0" xyz=" 0.175  0.175 0" rpy="3.141 0 -0.7854"/>
+    <xacro:flex_arm prefix="arm2" L="0.3" n="10" m="1.0" xyz=" 0.175 -0.175 0" rpy="3.141 0 -2.3562"/>
+    <xacro:flex_arm prefix="arm3" L="0.3" n="10" m="1.0" xyz="-0.175 -0.175 0" rpy="3.141 0 2.3562"/>
+    <xacro:flex_arm prefix="arm4" L="0.3" n="10" m="1.0" xyz="-0.175  0.175 0" rpy="3.141 0 0.7854"/>
     <joint name="arm1_joint" type="fixed">
         <parent link="drone_base"/>

Commit message: Add baseline controller

File: assets/drone.xacro (robot description, xacro)
@@ -7,5 +7,5 @@
     <xacro:property name="arm_x" value="0.175"/>
     <xacro:property name="arm_y" value="0.175"/>
-    <xacro:property name="m" value="10.0" />
+    <xacro:property name="m" value="2.0" />
     <xacro:macro name="box_inertia" params="l1 l2 l3 mass">
         <inertia ixx="${1/12*mass*(l3*l3 + l1*l1)}" ixy="0.0" ixz="0.0"

File: assets/drone_w_arms.urdf (robot description, URDF)
Before this commit: robot drone_w_arms, 57 links, 56 joints
Links:
- link drone_base: mass 10.0 -> 2.0
Joints:
- joint x_pos: limit lower=-1000 upper=1000 effort=1000 velocity=1000 -> lower=-1000 upper=1000 effort=10000 velocity=10000
- joint y_pos: limit lower=-1000 upper=1000 effort=1000 velocity=1000 -> lower=-1000 upper=1000 effort=10000 velocity=10000
- joint z_pos: limit lower=-1000 upper=1000 effort=1000 velocity=1000 -> lower=-1000 upper=1000 effort=10000 velocity=10000

File: assets/drone_w_arms.xacro (robot description, xacro)
@@ -3,4 +3,6 @@
     <xacro:property name="min_ax" value="-1000"/>
     <xacro:property name="max_ax" value="1000"/>
+    <xacro:property name="max_effort" value="10000"/>
+    <xacro:property name="max_velocity" value="10000"/>
     <!-- Include the robot macro -->
     <xacro:include filename="drone.xacro"/>
@@ -17,5 +19,5 @@
         <child link="p1" />
         <axis xyz="1 0 0"/>
-        <limit lower="${min_ax}" upper="${max_ax}" effort="1000" velocity="1000"/>
+        <limit lower="${min_ax}" upper="${max_ax}" effort="${max_effort}" velocity="${max_velocity}"/>
     </joint>
     <joint name="y_pos" type="prismatic">
@@ -23,5 +25,5 @@
         <child link="p2" />
         <axis xyz="0 1 0"/>
-        <limit lower="${min_ax}" upper="${max_ax}" effort="1000" velocity="1000"/>
+        <limit lower="${min_ax}" upper="${max_ax}" effort="${max_effort}" velocity="${max_velocity}"/>
     </joint>
     <joint name="z_pos" type="prismatic">
@@ -29,5 +31,5 @@
         <child link="p3" />
         <axis xyz="0 0 1"/>
-        <limit lower="${min_ax}" upper="${max_ax}" effort="1000" velocity="1000"/>
+        <limit lower="${min_ax}" upper="${max_ax}" effort="${max_effort}" velocity="${max_velocity}"/>
     </joint>
     <joint name="base_joint" type="continuous">

Commit message: Update meshes

File: assets/drone.xacro (robot description, xacro)
@@ -2,6 +2,6 @@
 <robot xmlns:xacro="http://www.ros.org/wiki/xacro">
     <xacro:property name="pi2" value="${pi * 0.5}" />
-    <xacro:property name="l1" value="0.525" />
-    <xacro:property name="l2" value="0.525" />
+    <xacro:property name="l1" value="0.45" />
+    <xacro:property name="l2" value="0.45" />
     <xacro:property name="l3" value="0.1" />
     <xacro:property name="arm_x" value="0.175"/>
@@ -17,7 +17,7 @@
         <link name="${prefix}_base">
             <visual>
-                <origin xyz="0 0 0" rpy="0 0 0"/>
+                <origin xyz="0 0 0" rpy="${pi2} 0 0"/>
                 <geometry>
-                    <mesh filename="./meshes/Holybro-X500-V2-no-landinggear-arm-attachments.dae"/>
+                    <mesh filename="./meshes/Holybro-X500-V2-no-landinggear.dae" scale="0.001 0.001 0.001"/>
                 </geometry>
             </visual>
@@ -25,5 +25,5 @@
                 <origin xyz="0 0 ${-l3*0.1}" rpy="0 0 0"/>
                 <geometry>
-                    <box size="${l1} ${l2} ${l3}"/>
+                    <cylinder radius="${sqrt(l1*l1 + l2*l2)/2}" length="${l3}"/>
                 </geometry>
             </collision>
@@ -36,5 +36,5 @@
         <link name="${prefix}_prop1">
             <visual>
-                <origin xyz="0 0 0" rpy="0 0 0"/>
+                <origin xyz="0 0 0.02" rpy="0 0 0"/>
                 <geometry>
                     <mesh filename="./meshes/1345_prop_ccw.dae" scale="0.75 0.75 0.75"/>
@@ -56,5 +56,5 @@
         <link name="${prefix}_prop2">
             <visual>
-                <origin xyz="0 0 0" rpy="0 0 0"/>
+                <origin xyz="0 0 0.02" rpy="0 0 0"/>
                 <geometry>
                     <mesh filename="./meshes/1345_prop_cw.dae" scale="0.75 0.75 0.75"/>
@@ -76,5 +76,5 @@
         <link name="${prefix}_prop3">
             <visual>
-                <origin xyz="0 0 0" rpy="0 0 0"/>
+                <origin xyz="0 0 0.02" rpy="0 0 0"/>
                 <geometry>
                     <mesh filename="./meshes/1345_prop_ccw.dae" scale="0.75 0.75 0.75"/>
@@ -96,5 +96,5 @@
         <link name="${prefix}_prop4">
             <visual>
-                <origin xyz="0 0 0" rpy="0 0 0"/>
+                <origin xyz="0 0 0.02" rpy="0 0 0"/>
                 <geometry>
                     <mesh filename="./meshes/1345_prop_cw.dae" scale="0.75 0.75 0.75"/>

File: assets/drone_w_arms.urdf (robot description, URDF)
Before this commit: robot drone_w_arms, 57 links, 56 joints
Links:
- link drone_base: geometry collision cylinder length=0.1 radius=0.31819805153394637; visual mesh filename=./meshes/Holybro-X500-V2-no-landinggear.dae scale=0.001 0.001 0.001

Commit message: Add option to edit damping to xarco

File: assets/drone.xacro (robot description, xacro)
@@ -25,5 +25,5 @@
                 <origin xyz="0 0 ${-l3*0.1}" rpy="0 0 0"/>
                 <geometry>
-                    <cylinder radius="${sqrt(l1*l1 + l2*l2)/2}" length="${l3}"/>
+                    <box size="${l1} ${l2} ${l3}"/>
                 </geometry>
             </collision>

File: assets/drone_w_arms.urdf (robot description, URDF)
Before this commit: robot drone_w_arms, 57 links, 56 joints
Links:
- link drone_base: geometry collision box size=0.45 0.45 0.1; visual mesh filename=./meshes/Holybro-X500-V2-no-landinggear.dae scale=0.001 0.001 0.001
Joints:
- joint base_joint: limit (none) -> lower=-1000 upper=1000 effort=10000 velocity=100.0
- joint x_pos: limit lower=-1000 upper=1000 effort=10000 velocity=10000 -> lower=-1000 upper=1000 effort=10000 velocity=100.0
- joint y_pos: limit lower=-1000 upper=1000 effort=10000 velocity=10000 -> lower=-1000 upper=1000 effort=10000 velocity=100.0
- joint z_pos: limit lower=-1000 upper=1000 effort=10000 velocity=10000 -> lower=-1000 upper=1000 effort=10000 velocity=100.0

File: assets/drone_w_arms.xacro (robot description, xacro)
@@ -4,5 +4,7 @@
     <xacro:property name="max_ax" value="1000"/>
     <xacro:property name="max_effort" value="10000"/>
-    <xacro:property name="max_velocity" value="10000"/>
+    <xacro:property name="max_velocity" value="100.0"/>
+    <xacro:property name="lin_damping" value="0"/>
+    <xacro:property name="rot_damping" value="0"/>
     <!-- Include the robot macro -->
     <xacro:include filename="drone.xacro"/>
@@ -19,4 +21,5 @@
         <child link="p1" />
         <axis xyz="1 0 0"/>
+        <dynamics damping="${lin_damping}" friction="0.0"/>
         <limit lower="${min_ax}" upper="${max_ax}" effort="${max_effort}" velocity="${max_velocity}"/>
     </joint>
@@ -25,4 +28,5 @@
         <child link="p2" />
         <axis xyz="0 1 0"/>
+        <dynamics damping="${lin_damping}" friction="0.0"/>
         <limit lower="${min_ax}" upper="${max_ax}" effort="${max_effort}" velocity="${max_velocity}"/>
     </joint>
@@ -31,4 +35,5 @@
         <child link="p3" />
         <axis xyz="0 0 1"/>
+        <dynamics damping="${lin_damping}" friction="0.0"/>
         <limit lower="${min_ax}" upper="${max_ax}" effort="${max_effort}" velocity="${max_velocity}"/>
     </joint>
@@ -37,5 +42,6 @@
         <child link="drone_base" />
         <axis xyz="0 0 1"/>
-        <dynamics damping="100.0" friction="0.0"/>
+        <dynamics damping="${rot_damping}" friction="0.0"/>
+        <limit lower="${min_ax}" upper="${max_ax}" effort="${max_effort}" velocity="${max_velocity}"/>
     </joint>
     <!-- Add dummy arms -->
