Commit message: Make urdf simple if no visualization

File: assets/drone.xacro (robot description, xacro)
@@ -17,7 +17,17 @@
         <link name="${prefix}_base">
             <visual>
-                <origin xyz="0 0 0" rpy="${pi2} 0 0"/>
+                <xacro:if value="$(arg full_visuals)">
+                    <origin xyz="0 0 0" rpy="${pi2} 0 0"/>
+                </xacro:if>
+                <xacro:unless value="$(arg full_visuals)">
+                    <origin xyz="0 0 ${-l3*0.1}" rpy="0 0 0"/>
+                </xacro:unless>
                 <geometry>
-                    <mesh filename="./meshes/Holybro-X500-V2-no-landinggear.dae" scale="0.001 0.001 0.001"/>
+                    <xacro:if value="$(arg full_visuals)">
+                        <mesh filename="./meshes/Holybro-X500-V2-no-landinggear.dae" scale="0.001 0.001 0.001"/>
+                    </xacro:if>
+                    <xacro:unless value="$(arg full_visuals)">
+                        <box size="${l1} ${l2} ${l3}"/>
+                    </xacro:unless>
                 </geometry>
             </visual>
@@ -36,7 +46,17 @@
         <link name="${prefix}_prop1">
             <visual>
-                <origin xyz="0 0 0.02" rpy="0 0 0"/>
+                <xacro:if value="$(arg full_visuals)">
+                    <origin xyz="0 0 0.02" rpy="0 0 0"/>
+                </xacro:if>
+                <xacro:unless value="$(arg full_visuals)">
+                    <origin xyz="0 0 0" rpy="0 0 0"/>
+                </xacro:unless>
                 <geometry>
-                    <mesh filename="./meshes/1345_prop_ccw.dae" scale="0.75 0.75 0.75"/>
+                    <xacro:if value="$(arg full_visuals)">
+                        <mesh filename="./meshes/1345_prop_ccw.dae" scale="0.75 0.75 0.75"/>
+                    </xacro:if>
+                    <xacro:unless value="$(arg full_visuals)">
+                        <cylinder radius="0.125" length="0.01"/>
+                    </xacro:unless>
                 </geometry>
             </visual>
@@ -56,7 +76,17 @@
         <link name="${prefix}_prop2">
             <visual>
-                <origin xyz="0 0 0.02" rpy="0 0 0"/>
+                <xacro:if value="$(arg full_visuals)">
+                    <origin xyz="0 0 0.02" rpy="0 0 0"/>
+                </xacro:if>
+                <xacro:unless value="$(arg full_visuals)">
+                    <origin xyz="0 0 0" rpy="0 0 0"/>
+                </xacro:unless>
                 <geometry>
-                    <mesh filename="./meshes/1345_prop_cw.dae" scale="0.75 0.75 0.75"/>
+                    <xacro:if value="$(arg full_visuals)">
+                        <mesh filename="./meshes/1345_prop_cw.dae" scale="0.75 0.75 0.75"/>
+                    </xacro:if>
+                    <xacro:unless value="$(arg full_visuals)">
+                        <cylinder radius="0.125" length="0.01"/>
+                    </xacro:unless>
                 </geometry>
             </visual>
@@ -76,7 +106,17 @@
         <link name="${prefix}_prop3">
             <visual>
-                <origin xyz="0 0 0.02" rpy="0 0 0"/>
+                <xacro:if value="$(arg full_visuals)">
+                    <origin xyz="0 0 0.02" rpy="0 0 0"/>
+                </xacro:if>
+                <xacro:unless value="$(arg full_visuals)">
+                    <origin xyz="0 0 0" rpy="0 0 0"/>
+                </xacro:unless>
                 <geometry>
-                    <mesh filename="./meshes/1345_prop_ccw.dae" scale="0.75 0.75 0.75"/>
+                    <xacro:if value="$(arg full_visuals)">
+                        <mesh filename="./meshes/1345_prop_ccw.dae" scale="0.75 0.75 0.75"/>
+                    </xacro:if>
+                    <xacro:unless value="$(arg full_visuals)">
+                        <cylinder radius="0.125" length="0.01"/>
+                    </xacro:unless>
                 </geometry>
             </visual>
@@ -96,7 +136,17 @@
         <link name="${prefix}_prop4">
             <visual>
-                <origin xyz="0 0 0.02" rpy="0 0 0"/>
+                <xacro:if value="$(arg full_visuals)">
+                    <origin xyz="0 0 0.02" rpy="0 0 0"/>
+                </xacro:if>
+                <xacro:unless value="$(arg full_visuals)">
+                    <origin xyz="0 0 0" rpy="0 0 0"/>
+                </xacro:unless>
                 <geometry>
-                    <mesh filename="./meshes/1345_prop_cw.dae" scale="0.75 0.75 0.75"/>
+                    <xacro:if value="$(arg full_visuals)">
+                        <mesh filename="./meshes/1345_prop_cw.dae" scale="0.75 0.75 0.75"/>
+                    </xacro:if>
+                    <xacro:unless value="$(arg full_visuals)">
+                        <cylinder radius="0.125" length="0.01"/>
+                    </xacro:unless>
                 </geometry>
             </visual>

File: assets/drone_w_arms.xacro (robot description, xacro)
@@ -1,4 +1,5 @@
 <?xml version="1.0"?>
 <robot xmlns:xacro="http://www.ros.org/wiki/xacro" name="drone_w_arms">
+    <xacro:arg name="full_visuals" default="true"/>
     <xacro:property name="min_ax" value="-1000"/>
     <xacro:property name="max_ax" value="1000"/>

File: assets/drone_w_arms_simple.urdf (robot description, URDF)
Before this commit: robot drone_w_arms, 57 links, 56 joints
Links:
- link arm1_link_1: geometry collision cylinder length=0.03 radius=0.01; visual cylinder length=0.03 radius=0.01
- link arm1_link_10: geometry collision cylinder length=0.03 radius=0.01; visual cylinder length=0.03 radius=0.01
- link arm1_link_2: geometry collision cylinder length=0.03 radius=0.01; visual cylinder length=0.03 radius=0.01
- link arm1_link_3: geometry collision cylinder length=0.03 radius=0.01; visual cylinder length=0.03 radius=0.01
- link arm1_link_4: geometry collision cylinder length=0.03 radius=0.01; visual cylinder length=0.03 radius=0.01
- link arm1_link_5: geometry collision cylinder length=0.03 radius=0.01; visual cylinder length=0.03 radius=0.01
- link arm1_link_6: geometry collision cylinder length=0.03 radius=0.01; visual cylinder length=0.03 radius=0.01
- link arm1_link_7: geometry collision cylinder length=0.03 radius=0.01; visual cylinder length=0.03 radius=0.01
- link arm1_link_8: geometry collision cylinder length=0.03 radius=0.01; visual cylinder length=0.03 radius=0.01
- link arm1_link_9: geometry collision cylinder length=0.03 radius=0.01; visual cylinder length=0.03 radius=0.01
- link arm2_link_1: geometry collision cylinder length=0.03 radius=0.01; visual cylinder length=0.03 radius=0.01
- link arm2_link_10: geometry collision cylinder length=0.03 radius=0.01; visual cylinder length=0.03 radius=0.01
- link arm2_link_2: geometry collision cylinder length=0.03 radius=0.01; visual cylinder length=0.03 radius=0.01
- link arm2_link_3: geometry collision cylinder length=0.03 radius=0.01; visual cylinder length=0.03 radius=0.01
- link arm2_link_4: geometry collision cylinder length=0.03 radius=0.01; visual cylinder length=0.03 radius=0.01
- link arm2_link_5: geometry collision cylinder length=0.03 radius=0.01; visual cylinder length=0.03 radius=0.01
- link arm2_link_6: geometry collision cylinder length=0.03 radius=0.01; visual cylinder length=0.03 radius=0.01
- link arm2_link_7: geometry collision cylinder length=0.03 radius=0.01; visual cylinder length=0.03 radius=0.01
- link arm2_link_8: geometry collision cylinder length=0.03 radius=0.01; visual cylinder length=0.03 radius=0.01
- link arm2_link_9: geometry collision cylinder length=0.03 radius=0.01; visual cylinder length=0.03 radius=0.01
- link arm3_link_1: geometry collision cylinder length=0.03 radius=0.01; visual cylinder length=0.03 radius=0.01
- link arm3_link_10: geometry collision cylinder length=0.03 radius=0.01; visual cylinder length=0.03 radius=0.01
- link arm3_link_2: geometry collision cylinder length=0.03 radius=0.01; visual cylinder length=0.03 radius=0.01
- link arm3_link_3: geometry collision cylinder length=0.03 radius=0.01; visual cylinder length=0.03 radius=0.01
- link arm3_link_4: geometry collision cylinder length=0.03 radius=0.01; visual cylinder length=0.03 radius=0.01
- link arm3_link_5: geometry collision cylinder length=0.03 radius=0.01; visual cylinder length=0.03 radius=0.01
- link arm3_link_6: geometry collision cylinder length=0.03 radius=0.01; visual cylinder length=0.03 radius=0.01
- link arm3_link_7: geometry collision cylinder length=0.03 radius=0.01; visual cylinder length=0.03 radius=0.01
- link arm3_link_8: geometry collision cylinder length=0.03 radius=0.01; visual cylinder length=0.03 radius=0.01
- link arm3_link_9: geometry collision cylinder length=0.03 radius=0.01; visual cylinder length=0.03 radius=0.01
- link arm4_link_1: geometry collision cylinder length=0.03 radius=0.01; visual cylinder length=0.03 radius=0.01
- link arm4_link_10: geometry collision cylinder length=0.03 radius=0.01; visual cylinder length=0.03 radius=0.01
- link arm4_link_2: geometry collision cylinder length=0.03 radius=0.01; visual cylinder length=0.03 radius=0.01
- link arm4_link_3: geometry collision cylinder length=0.03 radius=0.01; visual cylinder length=0.03 radius=0.01
- link arm4_link_4: geometry collision cylinder length=0.03 radius=0.01; visual cylinder length=0.03 radius=0.01
- link arm4_link_5: geometry collision cylinder length=0.03 radius=0.01; visual cylinder length=0.03 radius=0.01
- link arm4_link_6: geometry collision cylinder length=0.03 radius=0.01; visual cylinder length=0.03 radius=0.01
- link arm4_link_7: geometry collision cylinder length=0.03 radius=0.01; visual cylinder length=0.03 radius=0.01
- link arm4_link_8: geometry collision cylinder length=0.03 radius=0.01; visual cylinder length=0.03 radius=0.01
- link arm4_link_9: geometry collision cylinder length=0.03 radius=0.01; visual cylinder length=0.03 radius=0.01
- link drone_base: geometry collision box size=0.45 0.45 0.1; visual box size=0.45 0.45 0.1
- link drone_prop1: geometry collision cylinder length=0.01 radius=0.125; visual cylinder length=0.01 radius=0.125
- link drone_prop2: geometry collision cylinder length=0.01 radius=0.125; visual cylinder length=0.01 radius=0.125
- link drone_prop3: geometry collision cylinder length=0.01 radius=0.125; visual cylinder length=0.01 radius=0.125
- link drone_prop4: geometry collision cylinder length=0.01 radius=0.125; visual cylinder length=0.01 radius=0.125

File: assets/dummy_arm.xacro (robot description, xacro)
@@ -28,5 +28,10 @@
             <visual>
                 <geometry>
-                    <mesh filename="meshes/single_segment.dae" scale="0.0006 0.0006 ${0.003 / n}"/>
+                    <xacro:if value="$(arg full_visuals)">
+                        <mesh filename="meshes/single_segment.dae" scale="0.0006 0.0006 ${0.003 / n}"/>
+                    </xacro:if>
+                    <xacro:unless value="$(arg full_visuals)">
+                         <cylinder radius="${width}" length="${l}" />
+                    </xacro:unless>
                 </geometry>
                 <origin xyz="0 0 ${l / 2}" />
@@ -62,5 +67,10 @@
                 <visual>
                     <geometry>
-                        <mesh filename="meshes/single_segment.dae" scale="0.0006 0.0006 ${0.003 / N}"/>
+                        <xacro:if value="$(arg full_visuals)">
+                            <mesh filename="meshes/single_segment.dae" scale="0.0006 0.0006 ${0.003 / N}"/>
+                        </xacro:if>
+                        <xacro:unless value="$(arg full_visuals)">
+                            <cylinder radius="${width}" length="${l}" />
+                        </xacro:unless>
                     </geometry>
                     <origin xyz="0 0 ${l / 2}" />

Commit message: Fix issue with dones not as np arrays

File: assets/drone.xacro (robot description, xacro)
@@ -2,6 +2,6 @@
 <robot xmlns:xacro="http://www.ros.org/wiki/xacro">
     <xacro:property name="pi2" value="${pi * 0.5}" />
-    <xacro:property name="l1" value="0.45" />
-    <xacro:property name="l2" value="0.45" />
+    <xacro:property name="l1" value="0.35" />
+    <xacro:property name="l2" value="0.35" />
     <xacro:property name="l3" value="0.1" />
     <xacro:property name="arm_x" value="0.175"/>
@@ -64,5 +64,5 @@
                 <origin xyz="0 0 0" rpy="0 0 0"/>
                 <geometry>
-                    <cylinder radius="0.125" length="0.01"/>
+                    <cylinder radius="0.025" length="0.01"/>
                 </geometry>
             </collision>
@@ -94,5 +94,5 @@
                 <origin xyz="0 0 0" rpy="0 0 0"/>
                 <geometry>
-                    <cylinder radius="0.125" length="0.01"/>
+                    <cylinder radius="0.025" length="0.01"/>
                 </geometry>
             </collision>
@@ -124,5 +124,5 @@
                 <origin xyz="0 0 0" rpy="0 0 0"/>
                 <geometry>
-                    <cylinder radius="0.125" length="0.01"/>
+                    <cylinder radius="0.025" length="0.01"/>
                 </geometry>
             </collision>
@@ -154,5 +154,5 @@
                 <origin xyz="0 0 0" rpy="0 0 0"/>
                 <geometry>
-                    <cylinder radius="0.125" length="0.01"/>
+                    <cylinder radius="0.025" length="0.01"/>
                 </geometry>
             </collision>

File: assets/drone_w_arms.urdf (robot description, URDF)
Before this commit: robot drone_w_arms, 57 links, 56 joints
Links:
- link drone_base: geometry collision box size=0.35 0.35 0.1; visual mesh filename=./meshes/Holybro-X500-V2-no-landinggear.dae scale=0.001 0.001 0.001
- link drone_prop1: geometry collision cylinder length=0.01 radius=0.025; visual mesh filename=./meshes/1345_prop_ccw.dae scale=0.75 0.75 0.75
- link drone_prop2: geometry collision cylinder length=0.01 radius=0.025; visual mesh filename=./meshes/1345_prop_cw.dae scale=0.75 0.75 0.75
- link drone_prop3: geometry collision cylinder length=0.01 radius=0.025; visual mesh filename=./meshes/1345_prop_ccw.dae scale=0.75 0.75 0.75
- link drone_prop4: geometry collision cylinder length=0.01 radius=0.025; visual mesh filename=./meshes/1345_prop_cw.dae scale=0.75 0.75 0.75

File: assets/drone_w_arms_simple.urdf (robot description, URDF)
Before this commit: robot drone_w_arms, 57 links, 56 joints
Links:
- link drone_base: geometry collision box size=0.35 0.35 0.1; visual box size=0.35 0.35 0.1
- link drone_prop1: geometry collision cylinder length=0.01 radius=0.025; visual cylinder length=0.01 radius=0.125
- link drone_prop2: geometry collision cylinder length=0.01 radius=0.025; visual cylinder length=0.01 radius=0.125
- link drone_prop3: geometry collision cylinder length=0.01 radius=0.025; visual cylinder length=0.01 radius=0.125
- link drone_prop4: geometry collision cylinder length=0.01 radius=0.025; visual cylinder length=0.01 radius=0.125
